File: EAGLE-Files/DPad-Buttons.brd (EAGLE design)
At the start: 49.5 x 31.8 mm, 1 part

Commit message: Updated board layout
Parts:
- moved JP1 7.62 mm to (50.8, 24.1)
Routing:
- net BUT4: track 81.0 -> 86.6 mm
- net BUT3: track 59.4 -> 64.7 mm
- net BUT2: track 48.8 -> 53.1 mm
- net BUT1: track 60.0 -> 56.8 mm
Other:
- outline, holes or cut-outs redrawn
Changed lines of the file:
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@@
 <board>
 <plain>
-<wire x1="49.53" y1="7.62" x2="43.18" y2="0" width="0" layer="20"/>
-<wire x1="43.18" y1="0" x2="6.35" y2="0" width="0" layer="20"/>
+<wire x1="49.53" y1="17.78" x2="26.67" y2="0" width="0" layer="20"/>
+<wire x1="26.67" y1="0" x2="6.35" y2="0" width="0" layer="20"/>
 <wire x1="6.35" y1="0" x2="0.02" y2="8.89" width="0" layer="20"/>
 <wire x1="0.02" y1="8.89" x2="0.02" y2="19.99" width="0" layer="20"/>
 <wire x1="0.02" y1="19.99" x2="10.16" y2="31.75" width="0" layer="20"/>
 <wire x1="10.16" y1="31.75" x2="27.61" y2="31.75" width="0" layer="20"/>
-<wire x1="27.61" y1="31.75" x2="49.53" y2="25.07" width="0" layer="20"/>
-<wire x1="49.53" y1="25.07" x2="49.53" y2="7.62" width="0" layer="20"/>
+<wire x1="27.61" y1="31.75" x2="49.53" y2="31.42" width="0" layer="20"/>
+<wire x1="49.53" y1="31.42" x2="49.53" y2="17.78" width="0" layer="20"/>
 <dimension x1="0" y1="34.29" x2="49.53" y2="34.29" x3="24.765" y3="39.37" textsize="1.778" layer="1"/>
 <dimension x1="52.07" y1="34.29" x2="52.07" y2="0" x3="58.42" y3="17.145" textsize="1.778" layer="1"/>
@@
 <hole x="27.94" y="31.75" drill="0.35"/>
 <hole x="30.48" y="31.75" drill="0.35"/>
-<hole x="31.75" y="30.48" drill="0.35"/>
-<hole x="34.29" y="30.48" drill="0.35"/>
-<hole x="35.56" y="29.21" drill="0.35"/>
-<hole x="38.1" y="29.21" drill="0.35"/>
-<hole x="39.37" y="27.94" drill="0.35"/>
-<hole x="41.91" y="27.94" drill="0.35"/>
-<hole x="43.18" y="26.67" drill="0.35"/>
-<hole x="45.72" y="26.67" drill="0.35"/>
-<hole x="46.99" y="25.4" drill="0.35"/>
+<hole x="33.02" y="31.75" drill="0.35"/>
+<hole x="35.56" y="31.75" drill="0.35"/>
+<hole x="38.1" y="31.75" drill="0.35"/>
+<hole x="40.64" y="31.75" drill="0.35"/>
+<hole x="43.18" y="31.75" drill="0.35"/>
+<hole x="45.72" y="31.75" drill="0.35"/>
+<hole x="48.26" y="31.75" drill="0.35"/>
+<hole x="49.53" y="30.48" drill="0.35"/>
+<hole x="49.53" y="27.94" drill="0.35"/>
 <hole x="49.53" y="25.4" drill="0.35"/>
 <hole x="49.53" y="22.86" drill="0.35"/>
 <hole x="49.53" y="20.32" drill="0.35"/>
 <hole x="49.53" y="17.78" drill="0.35"/>
-<hole x="49.53" y="15.24" drill="0.35"/>
-<hole x="49.53" y="12.7" drill="0.35"/>
-<hole x="49.53" y="10.16" drill="0.35"/>
-<hole x="49.53" y="7.62" drill="0.35"/>
-<hole x="48.26" y="6.35" drill="0.35"/>
-<hole x="46.99" y="5.08" drill="0.35"/>
-<hole x="45.72" y="3.81" drill="0.35"/>
-<hole x="44.45" y="2.54" drill="0.35"/>
-<hole x="43.18" y="1.27" drill="0.35"/>
-<hole x="41.91" y="0" drill="0.35"/>
-<hole x="39.37" y="0" drill="0.35"/>
-<hole x="36.83" y="0" drill="0.35"/>
-<hole x="34.29" y="0" drill="0.35"/>
-<hole x="31.75" y="0" drill="0.35"/>
-<hole x="29.21" y="0" drill="0.35"/>
+<hole x="33.02" y="5.08" drill="0.35"/>
+<hole x="31.75" y="3.81" drill="0.35"/>
+<hole x="30.48" y="2.54" drill="0.35"/>
+<hole x="29.21" y="1.27" drill="0.35"/>
 <hole x="26.67" y="0" drill="0.35"/>
 <hole x="24.13" y="0" drill="0.35"/>
@@
 <hole x="7.62" y="29.21" drill="0.35"/>
 <hole x="8.89" y="30.48" drill="0.35"/>
+<hole x="34.29" y="6.35" drill="0.35"/>
+<hole x="35.56" y="7.62" drill="0.35"/>
+<hole x="36.83" y="8.89" drill="0.35"/>
+<hole x="38.1" y="8.89" drill="0.35"/>
+<hole x="39.37" y="10.16" drill="0.35"/>
+<hole x="40.64" y="11.43" drill="0.35"/>
+<hole x="41.91" y="12.7" drill="0.35"/>
+<hole x="43.18" y="13.97" drill="0.35"/>
+<hole x="44.45" y="13.97" drill="0.35"/>
+<hole x="45.72" y="15.24" drill="0.35"/>
+<hole x="46.99" y="16.51" drill="0.35"/>
+<hole x="48.26" y="16.51" drill="0.35"/>
 </plain>
 <attributes>
@@
 </autorouter>
 <elements>
-<element name="JP1" library="pinhead" library_urn="urn:adsk.eagle:library:325" package="1X05/90" package3d_urn="urn:adsk.eagle:package:22467/2" value="" x="50.8" y="16.51" smashed="yes" rot="R270">
-<attribute name="NAME" x="46.99" y="23.495" size="1.27" layer="25" ratio="10"/>
-<attribute name="POPULARITY" value="9" x="44.45" y="-3.81" size="1.778" layer="27" rot="R270" display="off"/>
-<attribute name="VALUE" x="46.99" y="8.255" size="1.27" layer="27"/>
+<element name="JP1" library="pinhead" library_urn="urn:adsk.eagle:library:325" package="1X05/90" package3d_urn="urn:adsk.eagle:package:22467/2" value="" x="50.8" y="24.13" smashed="yes" rot="R270">
+<attribute name="NAME" x="46.99" y="31.115" size="1.27" layer="25" ratio="10"/>
+<attribute name="POPULARITY" value="9" x="44.45" y="3.81" size="1.778" layer="27" rot="R270" display="off"/>
+<attribute name="VALUE" x="46.99" y="15.875" size="1.27" layer="27"/>
 </element>
 </elements>
@@
 <wire x1="15.113" y1="25.273" x2="15.113" y2="28.702" width="0.1524" layer="16"/>
 <wire x1="15.113" y1="28.702" x2="22.606" y2="28.702" width="0.1524" layer="16"/>
-<wire x1="25.1333" y1="28.2067" x2="22.606" y2="28.2067" width="0.635" layer="16"/>
-<wire x1="46.99" y1="19.05" x2="34.29" y2="19.05" width="0.635" layer="16"/>
-<wire x1="34.29" y1="19.05" x2="25.1333" y2="28.2067" width="0.635" layer="16"/>
+<wire x1="46.99" y1="26.67" x2="45.72" y2="26.67" width="0.635" layer="16"/>
+<wire x1="45.72" y1="26.67" x2="44.1833" y2="28.2067" width="0.635" layer="16"/>
+<wire x1="44.1833" y1="28.2067" x2="22.606" y2="28.2067" width="0.635" layer="16"/>
 </signal>
 <signal name="BUT2">
@@
 <wire x1="27.178" y1="14.478" x2="26.543" y2="14.478" width="0.1524" layer="16"/>
 <wire x1="26.543" y1="14.478" x2="26.543" y2="20.447" width="0.1524" layer="16"/>
-<wire x1="26.543" y1="20.447" x2="29.972" y2="20.447" width="0.1524" layer="16"/>
-<wire x1="29.972" y1="20.447" x2="29.972" y2="16.51" width="0.1524" layer="16"/>
-<wire x1="29.972" y1="16.51" x2="29.972" y2="12.954" width="0.1524" layer="16"/>
-<wire x1="46.99" y1="16.51" x2="29.972" y2="16.51" width="0.635" layer="16"/>
+<wire x1="26.543" y1="20.447" x2="27.94" y2="20.447" width="0.1524" layer="16"/>
+<wire x1="27.94" y1="20.447" x2="29.972" y2="20.447" width="0.1524" layer="16"/>
+<wire x1="29.972" y1="20.447" x2="29.972" y2="12.954" width="0.1524" layer="16"/>
+<wire x1="46.99" y1="24.13" x2="30.48" y2="24.13" width="0.635" layer="16"/>
+<wire x1="30.48" y1="24.13" x2="27.94" y2="21.59" width="0.635" layer="16"/>
+<wire x1="27.94" y1="21.59" x2="27.94" y2="20.447" width="0.635" layer="16"/>
 </signal>
 <signal name="BUT3">
@@
 <wire x1="22.606" y1="6.35" x2="22.606" y2="4.826" width="0.1524" layer="16"/>
 <wire x1="22.606" y1="4.826" x2="15.113" y2="4.826" width="0.1524" layer="16"/>
-<wire x1="46.99" y1="13.97" x2="43.18" y2="13.97" width="0.635" layer="16"/>
-<wire x1="43.18" y1="13.97" x2="35.56" y2="6.35" width="0.635" layer="16"/>
-<wire x1="35.56" y1="6.35" x2="22.606" y2="6.35" width="0.635" layer="16"/>
+<wire x1="46.99" y1="21.59" x2="45.72" y2="21.59" width="0.635" layer="16"/>
+<wire x1="45.72" y1="21.59" x2="44.45" y2="20.32" width="0.635" layer="16"/>
+<wire x1="44.45" y1="20.32" x2="36.83" y2="20.32" width="0.635" layer="16"/>
+<wire x1="36.83" y1="20.32" x2="33.02" y2="16.51" width="0.635" layer="16"/>
+<wire x1="33.02" y1="16.51" x2="33.02" y2="12.7" width="0.635" layer="16"/>
+<wire x1="26.67" y1="6.35" x2="22.606" y2="6.35" width="0.635" layer="16"/>
+<wire x1="33.02" y1="12.7" x2="26.67" y2="6.35" width="0.635" layer="16"/>
 </signal>
 <signal name="BUT4">
@@
 <wire x1="8.89" y1="12.954" x2="7.366" y2="12.954" width="0.1524" layer="16"/>
 <wire x1="7.366" y1="12.954" x2="7.366" y2="20.447" width="0.1524" layer="16"/>
-<wire x1="46.99" y1="11.43" x2="38.1" y2="2.54" width="0.635" layer="16"/>
-<wire x1="38.1" y1="2.54" x2="13.97" y2="2.54" width="0.635" layer="16"/>
 <wire x1="13.97" y1="2.54" x2="8.89" y2="7.62" width="0.635" layer="16"/>
 <wire x1="8.89" y1="7.62" x2="8.89" y2="12.954" width="0.635" layer="16"/>
+<wire x1="46.99" y1="19.05" x2="37.719" y2="19.05" width="0.635" layer="16"/>
+<wire x1="37.719" y1="19.05" x2="34.29" y2="15.621" width="0.635" layer="16"/>
+<wire x1="34.29" y1="11.43" x2="25.4" y2="2.54" width="0.635" layer="16"/>
+<wire x1="25.4" y1="2.54" x2="13.97" y2="2.54" width="0.635" layer="16"/>
+<wire x1="34.29" y1="15.621" x2="34.29" y2="11.43" width="0.635" layer="16"/>
 </signal>
 <signal name="EBUT1">
