File: EAGLE-Files/Four-Buttons.brd (EAGLE design)
At the start: 49.5 x 31.8 mm, 1 part

Commit message: Updated board layout
Parts:
- moved JP1 7.62 mm to (0.00, 24.1)
Routing:
- net BUT1: track 57.7 -> 65.3 mm
- net BUT2: track 70.6 -> 77.3 mm
- net BUT3: track 41.7 -> 44.3 mm
Other:
- outline, holes or cut-outs redrawn
Changed lines of the file:
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@@
 <board>
 <plain>
-<wire x1="0" y1="7.62" x2="6.35" y2="0" width="0" layer="20"/>
-<wire x1="6.35" y1="0" x2="43.18" y2="0" width="0" layer="20"/>
+<wire x1="0" y1="17.78" x2="17.78" y2="0" width="0" layer="20"/>
+<wire x1="17.78" y1="0" x2="43.18" y2="0" width="0" layer="20"/>
 <wire x1="43.18" y1="0" x2="49.51" y2="8.89" width="0" layer="20"/>
 <wire x1="49.51" y1="8.89" x2="49.51" y2="19.99" width="0" layer="20"/>
 <wire x1="49.51" y1="19.99" x2="39.37" y2="31.75" width="0" layer="20"/>
 <wire x1="39.37" y1="31.75" x2="21.92" y2="31.75" width="0" layer="20"/>
-<wire x1="21.92" y1="31.75" x2="0" y2="25.07" width="0" layer="20"/>
-<wire x1="0" y1="25.07" x2="0" y2="7.62" width="0" layer="20"/>
+<wire x1="21.92" y1="31.75" x2="0" y2="31.42" width="0" layer="20"/>
+<wire x1="0" y1="31.42" x2="0" y2="17.78" width="0" layer="20"/>
 <dimension x1="24.13" y1="27.94" x2="24.13" y2="5.08" x3="21.59" y3="16.51" textsize="1.778" layer="1"/>
 <dimension x1="16.51" y1="21.59" x2="41.91" y2="21.59" x3="29.21" y3="31.75" textsize="1.778" layer="1"/>
 <hole x="0" y="25.4" drill="0.35"/>
-<hole x="2.54" y="26.67" drill="0.35"/>
-<hole x="5.08" y="26.67" drill="0.35"/>
-<hole x="7.62" y="27.94" drill="0.35"/>
-<hole x="10.16" y="27.94" drill="0.35"/>
-<hole x="12.7" y="29.21" drill="0.35"/>
-<hole x="15.24" y="29.21" drill="0.35"/>
-<hole x="17.78" y="30.48" drill="0.35"/>
-<hole x="20.32" y="30.48" drill="0.35"/>
+<hole x="11.43" y="31.75" drill="0.35"/>
+<hole x="13.97" y="31.75" drill="0.35"/>
+<hole x="16.51" y="31.75" drill="0.35"/>
+<hole x="19.05" y="31.75" drill="0.35"/>
 <hole x="21.59" y="31.75" drill="0.35"/>
 <hole x="24.13" y="31.75" drill="0.35"/>
@@
 <hole x="20.32" y="0" drill="0.35"/>
 <hole x="17.78" y="0" drill="0.35"/>
-<hole x="15.24" y="0" drill="0.35"/>
-<hole x="12.7" y="0" drill="0.35"/>
-<hole x="10.16" y="0" drill="0.35"/>
-<hole x="7.62" y="0" drill="0.35"/>
-<hole x="5.08" y="1.27" drill="0.35"/>
-<hole x="3.81" y="2.54" drill="0.35"/>
-<hole x="2.54" y="3.81" drill="0.35"/>
-<hole x="1.27" y="5.08" drill="0.35"/>
-<hole x="0" y="6.35" drill="0.35"/>
-<hole x="0" y="8.89" drill="0.35"/>
-<hole x="0" y="11.43" drill="0.35"/>
-<hole x="0" y="13.97" drill="0.35"/>
-<hole x="0" y="16.51" drill="0.35"/>
+<hole x="16.51" y="1.27" drill="0.35"/>
+<hole x="15.24" y="2.54" drill="0.35"/>
+<hole x="13.97" y="3.81" drill="0.35"/>
+<hole x="12.7" y="5.08" drill="0.35"/>
+<hole x="11.43" y="6.35" drill="0.35"/>
+<hole x="10.16" y="7.62" drill="0.35"/>
+<hole x="2.54" y="15.24" drill="0.35"/>
+<hole x="1.27" y="16.51" drill="0.35"/>
 <hole x="0" y="19.05" drill="0.35"/>
 <hole x="0" y="21.59" drill="0.35"/>
@@
 <dimension x1="0" y1="34.29" x2="49.53" y2="34.29" x3="24.765" y3="39.37" textsize="1.778" layer="1"/>
 <dimension x1="52.07" y1="34.29" x2="52.07" y2="0" x3="58.42" y3="17.145" textsize="1.778" layer="1"/>
+<hole x="8.89" y="31.75" drill="0.35"/>
+<hole x="6.35" y="31.75" drill="0.35"/>
+<hole x="3.81" y="31.75" drill="0.35"/>
+<hole x="1.27" y="31.75" drill="0.35"/>
+<hole x="0" y="30.48" drill="0.35"/>
+<hole x="0" y="27.94" drill="0.35"/>
+<hole x="8.89" y="8.89" drill="0.35"/>
+<hole x="7.62" y="10.16" drill="0.35"/>
+<hole x="6.35" y="11.43" drill="0.35"/>
+<hole x="5.08" y="12.7" drill="0.35"/>
+<hole x="3.81" y="13.97" drill="0.35"/>
 </plain>
 <attributes>
@@
 </autorouter>
 <elements>
-<element name="JP1" library="pinhead" library_urn="urn:adsk.eagle:library:325" package="1X05/90" package3d_urn="urn:adsk.eagle:package:22467/2" value="" x="0" y="16.51" smashed="yes" rot="R90">
-<attribute name="NAME" x="3.81" y="9.525" size="1.27" layer="25" ratio="10" rot="R180"/>
-<attribute name="POPULARITY" value="9" x="6.35" y="36.83" size="1.778" layer="27" rot="R90" display="off"/>
-<attribute name="VALUE" x="3.81" y="24.765" size="1.27" layer="27" rot="R180"/>
+<element name="JP1" library="pinhead" library_urn="urn:adsk.eagle:library:325" package="1X05/90" package3d_urn="urn:adsk.eagle:package:22467/2" value="" x="0" y="24.13" smashed="yes" rot="R90">
+<attribute name="NAME" x="3.81" y="17.145" size="1.27" layer="25" ratio="10" rot="R180"/>
+<attribute name="POPULARITY" value="9" x="6.35" y="44.45" size="1.778" layer="27" rot="R90" display="off"/>
+<attribute name="VALUE" x="3.81" y="32.385" size="1.27" layer="27" rot="R180"/>
 </element>
 </elements>
@@
 <vertex x="32.766" y="3.556"/>
 </polygon>
-<wire x1="25.273" y1="3.556" x2="25.273" y2="4.191" width="0.1524" layer="16"/>
+<wire x1="25.273" y1="3.556" x2="25.273" y2="3.81" width="0.1524" layer="16"/>
+<wire x1="25.273" y1="3.81" x2="25.273" y2="4.191" width="0.1524" layer="16"/>
 <wire x1="25.273" y1="4.191" x2="31.623" y2="4.191" width="0.1524" layer="16"/>
 <wire x1="31.623" y1="4.191" x2="32.004" y2="4.572" width="0.1524" layer="16"/>
@@
 <wire x1="26.797" y1="6.985" x2="32.766" y2="6.985" width="0.1524" layer="16"/>
 <wire x1="32.766" y1="6.985" x2="32.766" y2="3.556" width="0.1524" layer="16"/>
-<wire x1="32.766" y1="3.556" x2="25.4" y2="3.556" width="0.1524" layer="16"/>
-<wire x1="25.4" y1="3.556" x2="25.273" y2="3.556" width="0.1524" layer="16"/>
-<wire x1="3.81" y1="13.97" x2="5.08" y2="13.97" width="0.635" layer="16"/>
-<wire x1="15.494" y1="3.556" x2="25.4" y2="3.556" width="0.635" layer="16"/>
-<wire x1="5.08" y1="13.97" x2="15.494" y2="3.556" width="0.635" layer="16"/>
+<wire x1="32.766" y1="3.556" x2="25.273" y2="3.556" width="0.1524" layer="16"/>
+<wire x1="3.81" y1="21.59" x2="6.35" y2="21.59" width="0.635" layer="16"/>
+<wire x1="10.287" y1="17.653" x2="10.287" y2="12.22655" width="0.635" layer="16"/>
+<wire x1="10.287" y1="12.22655" x2="13.62355" y2="8.89" width="0.635" layer="16"/>
+<wire x1="13.62355" y1="8.89" x2="21.59" y2="8.89" width="0.635" layer="16"/>
+<wire x1="21.59" y1="8.89" x2="22.86" y2="7.62" width="0.635" layer="16"/>
+<wire x1="22.86" y1="7.62" x2="22.86" y2="5.08" width="0.635" layer="16"/>
+<wire x1="22.86" y1="5.08" x2="24.13" y2="3.81" width="0.635" layer="16"/>
+<wire x1="24.13" y1="3.81" x2="25.273" y2="3.81" width="0.635" layer="16"/>
+<wire x1="6.35" y1="21.59" x2="10.287" y2="17.653" width="0.635" layer="16"/>
 </signal>
 <signal name="BUT2">
@@
 <wire x1="42.545" y1="12.954" x2="39.116" y2="12.954" width="0.1524" layer="16"/>
 <wire x1="39.116" y1="12.954" x2="39.116" y2="20.447" width="0.1524" layer="16"/>
-<wire x1="3.81" y1="16.51" x2="5.08" y2="16.51" width="0.635" layer="16"/>
-<wire x1="5.08" y1="16.51" x2="11.049" y2="10.541" width="0.635" layer="16"/>
-<wire x1="11.049" y1="10.541" x2="36.703" y2="10.541" width="0.635" layer="16"/>
-<wire x1="36.703" y1="10.541" x2="39.116" y2="12.954" width="0.635" layer="16"/>
+<wire x1="3.81" y1="24.13" x2="5.54706875" y2="24.13" width="0.635" layer="16"/>
+<wire x1="5.54706875" y1="24.13" x2="11.43" y2="18.24706875" width="0.635" layer="16"/>
+<wire x1="11.43" y1="18.24706875" x2="11.43" y2="12.7" width="0.635" layer="16"/>
+<wire x1="11.43" y1="12.7" x2="13.97" y2="10.16" width="0.635" layer="16"/>
+<wire x1="13.97" y1="10.16" x2="36.322" y2="10.16" width="0.635" layer="16"/>
+<wire x1="36.322" y1="10.16" x2="39.116" y2="12.954" width="0.635" layer="16"/>
 </signal>
 <signal name="BUT3">
@@
 <wire x1="17.145" y1="18.923" x2="17.145" y2="12.954" width="0.1524" layer="16"/>
 <wire x1="17.145" y1="12.954" x2="13.716" y2="12.954" width="0.1524" layer="16"/>
-<wire x1="13.716" y1="12.954" x2="13.716" y2="19.05" width="0.1524" layer="16"/>
-<wire x1="13.716" y1="19.05" x2="13.716" y2="20.447" width="0.1524" layer="16"/>
-<wire x1="3.81" y1="19.05" x2="13.716" y2="19.05" width="0.635" layer="16"/>
+<wire x1="13.716" y1="12.954" x2="13.716" y2="20.32" width="0.1524" layer="16"/>
+<wire x1="13.716" y1="20.32" x2="13.716" y2="20.447" width="0.1524" layer="16"/>
+<wire x1="3.81" y1="26.67" x2="7.366" y2="26.67" width="0.635" layer="16"/>
+<wire x1="7.366" y1="26.67" x2="13.716" y2="20.32" width="0.635" layer="16"/>
 </signal>
 <signal name="BUT4">
@@
 <wire x1="32.766" y1="28.575" x2="32.766" y2="25.146" width="0.1524" layer="16"/>
 <wire x1="32.766" y1="25.146" x2="25.273" y2="25.146" width="0.1524" layer="16"/>
-<wire x1="3.81" y1="21.59" x2="7.62" y2="21.59" width="0.635" layer="16"/>
-<wire x1="11.43" y1="25.4" x2="25.273" y2="25.4" width="0.635" layer="16"/>
-<wire x1="7.62" y1="21.59" x2="11.43" y2="25.4" width="0.635" layer="16"/>
+<wire x1="25.273" y1="25.4" x2="24.13" y2="25.4" width="0.635" layer="16"/>
+<wire x1="24.13" y1="25.4" x2="20.32" y2="29.21" width="0.635" layer="16"/>
+<wire x1="20.32" y1="29.21" x2="3.81" y2="29.21" width="0.635" layer="16"/>
 </signal>
 <signal name="EBUT1">
