File: EAGLE-Files/Four-Buttons.brd (EAGLE design)
At the start: 49.5 x 31.8 mm, 1 part

Commit message: Updated board layouts
Parts:
- added JP2, JP3, JP4: (no value), pinhead:1X01
Connections:
- net GND: now also JP2.1, JP3.1, JP4.1
Routing:
- net BUT1: track 65.3 -> 66.8 mm
- net BUT2: track 77.3 -> 78.8 mm
Changed lines of the file:
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@@
 <attribute name="VALUE" x="3.81" y="32.385" size="1.27" layer="27" rot="R180"/>
+</element>
+<element name="JP2" library="pinhead" library_urn="urn:adsk.eagle:library:325" package="1X01" package3d_urn="urn:adsk.eagle:package:22485/2" value="" x="7.62" y="15.24" smashed="yes">
+<attribute name="NAME" x="6.2738" y="17.0688" size="1.27" layer="25" ratio="10"/>
+<attribute name="POPULARITY" value="64" x="7.62" y="15.24" size="1.778" layer="27" display="off"/>
+<attribute name="VALUE" x="6.35" y="12.065" size="1.27" layer="27"/>
+</element>
+<element name="JP3" library="pinhead" library_urn="urn:adsk.eagle:library:325" package="1X01" package3d_urn="urn:adsk.eagle:package:22485/2" value="" x="13.97" y="25.4" smashed="yes">
+<attribute name="NAME" x="12.6238" y="27.2288" size="1.27" layer="25" ratio="10"/>
+<attribute name="POPULARITY" value="64" x="13.97" y="25.4" size="1.778" layer="27" display="off"/>
+<attribute name="VALUE" x="12.7" y="22.225" size="1.27" layer="27"/>
+</element>
+<element name="JP4" library="pinhead" library_urn="urn:adsk.eagle:library:325" package="1X01" package3d_urn="urn:adsk.eagle:package:22485/2" value="" x="7.62" y="19.05" smashed="yes">
+<attribute name="NAME" x="6.2738" y="20.8788" size="1.27" layer="25" ratio="10"/>
+<attribute name="POPULARITY" value="64" x="7.62" y="19.05" size="1.778" layer="27" display="off"/>
+<attribute name="VALUE" x="6.35" y="15.875" size="1.27" layer="27"/>
 </element>
 </elements>
@@
 <vertex x="54.61" y="36.83"/>
 </polygon>
+<contactref element="JP2" pad="1"/>
+<contactref element="JP3" pad="1"/>
+<contactref element="JP4" pad="1"/>
 </signal>
 <signal name="BUT1">
@@
 <wire x1="32.766" y1="6.985" x2="32.766" y2="3.556" width="0.1524" layer="16"/>
 <wire x1="32.766" y1="3.556" x2="25.273" y2="3.556" width="0.1524" layer="16"/>
-<wire x1="3.81" y1="21.59" x2="6.35" y2="21.59" width="0.635" layer="16"/>
-<wire x1="10.287" y1="17.653" x2="10.287" y2="12.22655" width="0.635" layer="16"/>
+<wire x1="3.81" y1="21.59" x2="8.89" y2="21.59" width="0.635" layer="16"/>
+<wire x1="10.287" y1="20.193" x2="10.287" y2="12.22655" width="0.635" layer="16"/>
 <wire x1="10.287" y1="12.22655" x2="13.62355" y2="8.89" width="0.635" layer="16"/>
 <wire x1="13.62355" y1="8.89" x2="21.59" y2="8.89" width="0.635" layer="16"/>
@@
 <wire x1="22.86" y1="5.08" x2="24.13" y2="3.81" width="0.635" layer="16"/>
 <wire x1="24.13" y1="3.81" x2="25.273" y2="3.81" width="0.635" layer="16"/>
-<wire x1="6.35" y1="21.59" x2="10.287" y2="17.653" width="0.635" layer="16"/>
+<wire x1="8.89" y1="21.59" x2="10.287" y2="20.193" width="0.635" layer="16"/>
 </signal>
 <signal name="BUT2">
@@
 <wire x1="42.545" y1="12.954" x2="39.116" y2="12.954" width="0.1524" layer="16"/>
 <wire x1="39.116" y1="12.954" x2="39.116" y2="20.447" width="0.1524" layer="16"/>
-<wire x1="3.81" y1="24.13" x2="5.54706875" y2="24.13" width="0.635" layer="16"/>
-<wire x1="5.54706875" y1="24.13" x2="11.43" y2="18.24706875" width="0.635" layer="16"/>
-<wire x1="11.43" y1="18.24706875" x2="11.43" y2="12.7" width="0.635" layer="16"/>
+<wire x1="3.81" y1="24.13" x2="8.08706875" y2="24.13" width="0.635" layer="16"/>
+<wire x1="8.08706875" y1="24.13" x2="11.43" y2="20.78706875" width="0.635" layer="16"/>
+<wire x1="11.43" y1="20.78706875" x2="11.43" y2="12.7" width="0.635" layer="16"/>
 <wire x1="11.43" y1="12.7" x2="13.97" y2="10.16" width="0.635" layer="16"/>
 <wire x1="13.97" y1="10.16" x2="36.322" y2="10.16" width="0.635" layer="16"/>
