File: EAGLE-Files/Four-Buttons.sch (EAGLE design)
At the start: 1 part

Commit message: Updated board layouts
Parts:
- added JP2, JP3, JP4: (no value), pinhead:PINHD-1X1
Connections:
- net GND: now also JP2.1, JP3.1, JP4.1
Changed lines of the file:
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@@
 <part name="JP1" library="pinhead" library_urn="urn:adsk.eagle:library:325" deviceset="PINHD-1X5" device="/90" package3d_urn="urn:adsk.eagle:package:22467/2"/>
 <part name="GND1" library="supply1" library_urn="urn:adsk.eagle:library:371" deviceset="GND" device=""/>
+<part name="JP2" library="pinhead" library_urn="urn:adsk.eagle:library:325" deviceset="PINHD-1X1" device="" package3d_urn="urn:adsk.eagle:package:22485/2"/>
+<part name="GND2" library="supply1" library_urn="urn:adsk.eagle:library:371" deviceset="GND" device=""/>
+<part name="JP3" library="pinhead" library_urn="urn:adsk.eagle:library:325" deviceset="PINHD-1X1" device="" package3d_urn="urn:adsk.eagle:package:22485/2"/>
+<part name="GND3" library="supply1" library_urn="urn:adsk.eagle:library:371" deviceset="GND" device=""/>
+<part name="JP4" library="pinhead" library_urn="urn:adsk.eagle:library:325" deviceset="PINHD-1X1" device="" package3d_urn="urn:adsk.eagle:package:22485/2"/>
+<part name="GND4" library="supply1" library_urn="urn:adsk.eagle:library:371" deviceset="GND" device=""/>
 </parts>
 <sheets>
@@
 <attribute name="VALUE" x="71.12" y="50.8" size="1.778" layer="96" rot="R270"/>
 </instance>
+<instance part="JP2" gate="G$1" x="63.5" y="55.88" smashed="yes" rot="R90">
+<attribute name="NAME" x="60.325" y="49.53" size="1.778" layer="95" rot="R90"/>
+<attribute name="VALUE" x="68.58" y="49.53" size="1.778" layer="96" rot="R90"/>
+</instance>
+<instance part="GND2" gate="1" x="63.5" y="45.72" smashed="yes">
+<attribute name="VALUE" x="60.96" y="43.18" size="1.778" layer="96"/>
+</instance>
+<instance part="JP3" gate="G$1" x="55.88" y="55.88" smashed="yes" rot="R90">
+<attribute name="NAME" x="52.705" y="49.53" size="1.778" layer="95" rot="R90"/>
+<attribute name="VALUE" x="60.96" y="49.53" size="1.778" layer="96" rot="R90"/>
+</instance>
+<instance part="GND3" gate="1" x="55.88" y="45.72" smashed="yes">
+<attribute name="VALUE" x="53.34" y="43.18" size="1.778" layer="96"/>
+</instance>
+<instance part="JP4" gate="G$1" x="48.26" y="55.88" smashed="yes" rot="R90">
+<attribute name="NAME" x="45.085" y="49.53" size="1.778" layer="95" rot="R90"/>
+<attribute name="VALUE" x="53.34" y="49.53" size="1.778" layer="96" rot="R90"/>
+</instance>
+<instance part="GND4" gate="1" x="48.26" y="45.72" smashed="yes">
+<attribute name="VALUE" x="45.72" y="43.18" size="1.778" layer="96"/>
+</instance>
 </instances>
 <busses>
@@
 <wire x1="76.2" y1="48.26" x2="86.36" y2="48.26" width="0.1524" layer="91"/>
 </segment>
+<segment>
+<pinref part="JP2" gate="G$1" pin="1"/>
+<pinref part="GND2" gate="1" pin="GND"/>
+<wire x1="63.5" y1="53.34" x2="63.5" y2="48.26" width="0.1524" layer="91"/>
+</segment>
+<segment>
+<pinref part="JP3" gate="G$1" pin="1"/>
+<pinref part="GND3" gate="1" pin="GND"/>
+<wire x1="55.88" y1="53.34" x2="55.88" y2="48.26" width="0.1524" layer="91"/>
+</segment>
+<segment>
+<pinref part="JP4" gate="G$1" pin="1"/>
+<pinref part="GND4" gate="1" pin="GND"/>
+<wire x1="48.26" y1="53.34" x2="48.26" y2="48.26" width="0.1524" layer="91"/>
+</segment>
 </net>
